File: Grupos/1/PCB_Grupo_1.brd (EAGLE design)
At the start: 100 x 80 mm, 45 parts, among them T1 2N7002-7-F, T2 2N7002-7-F, U1 MAX3221ECPWR, U2 ST1S14PHR, U3 MAX31855KASA+T

Commit message: Revisión en progreso
Parts:
- R4: value 80.6 k -> 301K
- TP1, TP2, TP3, TP4: value (none) -> TEST_POINT
- renumbered T.P.1 to TP1, T.P.2 to TP2, T.P.3 to TP3, T.P.4 to TP4
Connections:
- net N$18 renamed 7.5V
- removed net N$20: CT3.4, M1.CN10-33, R7.1
- removed net N$21: M1.CN10-12, T1.G
- removed net N$23: D5.1, M1.CN10-21, R6.1
- removed net N$26: C11.1, M1.CN6-4, R7.2, R8.2, R9.2, U3.4
- removed net N$30: M1.CN10-28, U3.7
- removed net N$31: M1.CN10-16, U3.6
- removed net N$32: M1.CN10-30, U3.5
- removed net N$33: M1.CN10-35, U1.11
- removed net N$35: M1.CN10-37, U1.9
- removed net N$38: CT4.3, R10.1, TP2.P$1
- removed net N$39: D2.1, R14.1, TP4.P$1
- removed net N$8: C5.1, CT4.2, M1.CN6-5, U1.12, U1.15, U1.16
- new net +3.3V: C11.1, C5.1, M1.CN6-4, R7.2, R8.2, R9.2, U1.12, U1.15, U1.16, U3.4
- new net INPUT1: CT3.4, M1.CN8-1, R7.1
- new net INPUT2: D5.1, M1.CN8-4, R6.1
- new net MAX_CS: M1.CN5-3, U3.6
- new net MAX_SCK: M1.CN5-6, U3.5
- new net MAX_SO: M1.CN5-5, U3.7
- new net N$18: D2.1, R14.1, TP4.1
- new net OUTPUT1: M1.CN8-2, T2.G
- new net OUTPUT2: M1.CN8-3, T1.G
- new net RS232_DIN_MCU_TX: M1.CN5-1, U1.11
- new net RS232_ROUT_MCU_RX: M1.CN9-3, U1.9
- new net TP2: CT4.3, R10.1, TP2.1
- net N$15: now also TP1.1; no longer TP1.P$1
- net N$19: now also CT4.2, M1.CN6-5; no longer M1.CN10-14, T2.G
- net N$34: now also TP3.1; no longer TP3.P$1
- net N$36: now also M1.CN5-2; no longer M1.CN10-13
Routing:
- net N$21: track 129.8 -> 0.00 mm, vias 4 -> 0
- net N$8: track 123.1 -> 0.00 mm, vias 4 -> 0
- net TP2: track 0.00 -> 94.8 mm
- net N$38: track 94.8 -> 0.00 mm
- net +3.3V: track 0.00 -> 94.7 mm, vias 0 -> 4
- net N$20: track 94.4 -> 0.00 mm, vias 4 -> 0
- net N$26: track 71.4 -> 0.00 mm, vias 4 -> 0
- net N$19: track 55.2 -> 111.3 mm, vias 2 -> 0
- net INPUT1: track 0.00 -> 54.6 mm, vias 0 -> 2
- net RS232_DIN_MCU_TX: track 0.00 -> 49.9 mm, vias 0 -> 1
- net N$23: track 37.7 -> 0.00 mm, vias 2 -> 0
- net RS232_ROUT_MCU_RX: track 0.00 -> 36.2 mm, vias 0 -> 1
- net N$31: track 35.8 -> 0.00 mm
- net N$33: track 35.4 -> 0.00 mm
- net N$35: track 34.8 -> 0.00 mm
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