File: Grupos/1/PCB_Grupo_1.sch (EAGLE design)
At the start: 45 parts, among them T1 2N7002-7-F, T2 2N7002-7-F, U1 MAX3221ECPWR, U2 ST1S14PHR, U3 MAX31855KASA+T

Commit message: Revisión en progreso
Parts:
- removed T.P.1, T.P.2, T.P.3, T.P.4: (no value), TEST_POINT:TEST_POINT
- added TP1, TP2, TP3, TP4: TEST_POINT, TEST_POINT:TEST_POINT
- R4: value 80.6 k -> 301K; PART_NO RC0805FR-0780K6L -> RC0805FR-07301KL
- R8, R9: DNP (none) -> T
Connections:
- net N$18 renamed 7.5V
- removed net N$20: CT3.4, M1-CN10.PA10, R7.1
- removed net N$21: M1-CN10.PA12, T1.GATE
- removed net N$23: D5.C, M1-CN10.PA9, R6.1
- removed net N$26: C11.1, M1-CN6.+3V3, R7.2, R8.2, R9.2, U3.VCC
- removed net N$30: M1-CN10.PB14, U3.SO
- removed net N$31: M1-CN10.PB12, U3.CS'
- removed net N$32: M1-CN10.PB13, U3.SCK
- removed net N$33: M1-CN10.PA2, U1.DIN
- removed net N$35: M1-CN10.PA3, U1.ROUT
- removed net N$38: CT4.3, R10.1, T.P.2.T.P.
- removed net N$39: D2.C, R14.1, T.P.4.T.P.
- removed net N$8: C5.1, CT4.2, M1-CN6.+5V, U1.FORCEOFF, U1.FORCEON, U1.VCC
- new net +3.3V: C11.1, C5.1, M1-CN6.+3V3, R7.2, R8.2, R9.2, U1.FORCEOFF, U1.FORCEON, U1.VCC, U3.VCC
- new net INPUT1: CT3.4, M1-CN8.PA0, R7.1
- new net INPUT2: D5.C, M1-CN8.PB0, R6.1
- new net MAX_CS: M1-CN5.PB6, U3.CS'
- new net MAX_SCK: M1-CN5.PA5, U3.SCK
- new net MAX_SO: M1-CN5.PA6, U3.SO
- new net N$18: D2.C, R14.1, TP4.TP
- new net OUTPUT1: M1-CN8.PA1, T2.GATE
- new net OUTPUT2: M1-CN8.PA4, T1.GATE
- new net RS232_DIN_MCU_TX: M1-CN5.PA9, U1.DIN
- new net RS232_ROUT_MCU_RX: M1-CN9.PA10, U1.ROUT
- new net TP2: CT4.3, R10.1, TP2.TP
- net N$15: now also TP1.TP; no longer T.P.1.T.P.
- net N$19: now also CT4.2, M1-CN6.+5V; no longer M1-CN10.PA11, T2.GATE
- net N$34: now also TP3.TP; no longer T.P.3.T.P.
- net N$36: now also M1-CN5.PC7; no longer M1-CN10.PA6
