File: Grupos/13/Archivos_de_diseño/Esquematico.brd (EAGLE design)
At the start: 72.4 x 50.9 mm, 59 parts, among them J1 PH1-01-UA, J10 PH1-01-UA, J11 PH1-01-UA, J12 PH1-01-UA, J13 PH1-01-UA, J2 PH1-01-UA, J3 PH1-01-UA, J4 PH1-01-UA, J5 PH1-01-UA, J6 PH1-01-UA, J7 PH1-01-UA, J8 PH1-01-UA, J9 PH1-01-UA, U1 TLV7031QDBVRQ1, U10 TLV7031QDBVRQ1, U11 SN74AHC1G08DBVR, U12 SN74AHC1G08DBVR, U13 74LVC1G157GV-Q100H, U14 74LVC1G157GV-Q100H, U15 74LVC1G157GV-Q100H, U16 74LVC1G157GV-Q100H, U17 74LVC1G157GV-Q100H, U18 74LVC1G157GV-Q100H, U19 74LVC1G157GV-Q100H, U2 TLV7031QDBVRQ1, U20 74LVC1G157GV-Q100H, U21 CD74HC4002PWR, U3 TLV7031QDBVRQ1, U4 TLV7031QDBVRQ1, U5 TLV7031QDBVRQ1, U6 TLV7031QDBVRQ1, U7 TLV7031QDBVRQ1, U8 TLV7031QDBVRQ1, U9 TLV7031QDBVRQ1

Commit message: Se arregla librerías
Routing:
- net V3_O: track 54.5 -> 57.8 mm
- net -5V: track 150.7 -> 152.7 mm
- net N$37: track 53.1 -> 54.0 mm
- net V1_O: track 72.2 -> 72.8 mm
- net N$50: track 6.67 -> 7.27 mm
- net +5V: track 225.9 -> 226.4 mm
