File: Grupos/2/Review/Motor v2/motor_encoder.brd (EAGLE design)
At the start: 70.8 x 59.7 mm, 16 parts, among them U1 L9958SB, X1 1729128

Commit message: Se suben archivos posterior a revisión
Parts:
- VR1: value P160KN -> P160KN-0QD15B10K
Changed lines of the file:
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@@
 <element name="C1" library="rcl" library_urn="urn:adsk.eagle:library:334" package="C0805" package3d_urn="urn:adsk.eagle:package:23617/2" value="10nF" x="43.41" y="51.41" smashed="yes" rot="R180">
 <attribute name="NAME" x="44.18" y="50.14" size="1.2" layer="25" ratio="14" rot="R180"/>
+<attribute name="PARTNO" value="GRM2195C1H103JA01D" x="43.41" y="51.41" size="1.778" layer="27" rot="R180" display="off"/>
 <attribute name="POPULARITY" value="63" x="1.5" y="136.5" size="1.778" layer="27" rot="R180" display="off"/>
 <attribute name="SPICEPREFIX" value="C" x="1.5" y="136.5" size="1.778" layer="27" rot="R180" display="off"/>
@@
 <element name="C2" library="rcl" library_urn="urn:adsk.eagle:library:334" package="C0805" package3d_urn="urn:adsk.eagle:package:23617/2" value="10nF" x="48.74" y="51.59" smashed="yes">
 <attribute name="NAME" x="48.232" y="49.05" size="1.2" layer="25" ratio="14"/>
+<attribute name="PARTNO" value="GRM2195C1H103JA01D" x="48.74" y="51.59" size="1.778" layer="27" display="off"/>
 <attribute name="POPULARITY" value="63" x="97" y="-33.5" size="1.778" layer="27" display="off"/>
 <attribute name="SPICEPREFIX" value="C" x="97" y="-33.5" size="1.778" layer="27" display="off"/>
@@
 <element name="C3" library="rcl" library_urn="urn:adsk.eagle:library:334" package="C0805" package3d_urn="urn:adsk.eagle:package:23617/2" value="100nF" x="32.52" y="34.29" smashed="yes">
 <attribute name="NAME" x="31.631" y="32.004" size="1.2" layer="25" ratio="14"/>
+<attribute name="PARTNO" value="GCM21BR72A104KA37L" x="32.52" y="34.29" size="1.778" layer="27" display="off"/>
 <attribute name="POPULARITY" value="63" x="61.73" y="-50.8" size="1.778" layer="27" display="off"/>
 <attribute name="SPICEPREFIX" value="C" x="61.73" y="-50.8" size="1.778" layer="27" display="off"/>
@@
 <element name="C4" library="rcl" library_urn="urn:adsk.eagle:library:334" package="C0805" package3d_urn="urn:adsk.eagle:package:23617/2" value="1uF" x="27.94" y="34.29" smashed="yes" rot="R180">
 <attribute name="NAME" x="27.305" y="31.877" size="1.2" layer="25" ratio="14"/>
+<attribute name="PARTNO" value="GCJ219R71C105KA01D" x="27.94" y="34.29" size="1.778" layer="27" rot="R180" display="off"/>
 <attribute name="POPULARITY" value="63" x="-40.64" y="119.38" size="1.778" layer="27" rot="R180" display="off"/>
 <attribute name="SPICEPREFIX" value="C" x="-40.64" y="119.38" size="1.778" layer="27" rot="R180" display="off"/>
@@
 <element name="C5" library="rcl_v2" package="F80-UNITE_CHEMI-CON" value="100uF" x="29.98" y="40.64" smashed="yes" rot="R180">
 <attribute name="NAME" x="26.571" y="44.894" size="1.2" layer="25" ratio="14"/>
+<attribute name="PARTNO" value="EMVE250ADA101MF80G" x="29.98" y="40.64" size="1.778" layer="27" rot="R180" display="off"/>
 </element>
 <element name="C6" library="rcl" library_urn="urn:adsk.eagle:library:334" package="C0805" package3d_urn="urn:adsk.eagle:package:23617/2" value="100nF" x="40.44" y="33.59" smashed="yes">
 <attribute name="NAME" x="36.757" y="33.082" size="1.2" layer="25" ratio="14"/>
+<attribute name="PARTNO" value="GCM21BR72A104KA37L" x="40.44" y="33.59" size="1.778" layer="27" display="off"/>
 <attribute name="POPULARITY" value="63" x="76" y="-51.5" size="1.778" layer="27" display="off"/>
 <attribute name="SPICEPREFIX" value="C" x="76" y="-51.5" size="1.778" layer="27" display="off"/>
@@
 <element name="R1" library="rcl" library_urn="urn:adsk.eagle:library:334" package="R0805" package3d_urn="urn:adsk.eagle:package:23553/2" value="10K" x="36.09" y="42.84" smashed="yes" rot="R270">
 <attribute name="NAME" x="33.804" y="43.729" size="1.2" layer="25" ratio="14" rot="R270"/>
+<attribute name="PARTNO" value="RC0805FR-0710KL" x="36.09" y="42.84" size="1.778" layer="27" rot="R270" display="off"/>
 <attribute name="POPULARITY" value="85" x="-49" y="-10.5" size="1.778" layer="27" rot="R270" display="off"/>
 <attribute name="SPICEPREFIX" value="R" x="-49" y="-10.5" size="1.778" layer="27" rot="R270" display="off"/>
@@
 <element name="R2" library="rcl" library_urn="urn:adsk.eagle:library:334" package="R0805" package3d_urn="urn:adsk.eagle:package:23553/2" value="10K" x="37.08" y="47.59" smashed="yes">
 <attribute name="NAME" x="39.445" y="46.86" size="1.2" layer="25" ratio="14"/>
+<attribute name="PARTNO" value="RC0805FR-0710KL" x="37.08" y="47.59" size="1.778" layer="27" display="off"/>
 <attribute name="POPULARITY" value="85" x="95.5" y="-37.5" size="1.778" layer="27" display="off"/>
 <attribute name="SPICEPREFIX" value="R" x="95.5" y="-37.5" size="1.778" layer="27" display="off"/>
@@
 <element name="R3" library="rcl" library_urn="urn:adsk.eagle:library:334" package="R0805" package3d_urn="urn:adsk.eagle:package:23553/2" value="10K" x="51.57" y="47.26" smashed="yes" rot="R180">
 <attribute name="NAME" x="52.205" y="45.99" size="1.2" layer="25" ratio="14" rot="R180"/>
+<attribute name="PARTNO" value="RC0805FR-0710KL" x="51.57" y="47.26" size="1.778" layer="27" rot="R180" display="off"/>
 <attribute name="POPULARITY" value="85" x="-11.93" y="132.35" size="1.778" layer="27" rot="R180" display="off"/>
 <attribute name="SPICEPREFIX" value="R" x="-11.93" y="132.35" size="1.778" layer="27" rot="R180" display="off"/>
 <attribute name="VALUE" x="52.205" y="49.8" size="1.27" layer="27" rot="R180"/>
 </element>
-<element name="VR1" library="P160KN" package="P160KN-0QD15B10K" value="P160KN" x="29.21" y="5.08" smashed="yes" rot="R270">
+<element name="VR1" library="P160KN" package="P160KN-0QD15B10K" value="P160KN-0QD15B10K" x="29.21" y="5.08" smashed="yes" rot="R270">
 <attribute name="NAME" x="20.92" y="11.71" size="1.2" layer="25" ratio="14"/>
+<attribute name="PARTNO" value="P160KN-0QD15B10K" x="29.21" y="5.08" size="1.778" layer="27" rot="R270" display="off"/>
 </element>
-<element name="U1" library="L9958SBTR" package="POWERSO-16" value="L9958SB" x="45.72" y="40.64" smashed="yes" rot="R180"/>
+<element name="U1" library="L9958SBTR" package="POWERSO-16" value="L9958SB" x="45.72" y="40.64" smashed="yes" rot="R180">
+<attribute name="PARTNO" value="L9958SB" x="45.72" y="40.64" size="1.778" layer="27" rot="R180" display="off"/>
+</element>
 <element name="X1" library="1729128 - PHOENIX CONTACT" package="MKDSN1,5/2-5,08" package3d_urn="urn:adsk.eagle:package:9630/1" value="1729128" x="35.56" y="54.61" smashed="yes" rot="R180">
 <attribute name="NAME" x="28.962" y="55.3101" size="1.2" layer="25" ratio="14" rot="R270"/>
+<attribute name="PARTNO" value="1729128" x="35.56" y="54.61" size="1.778" layer="27" rot="R180" display="off"/>
 <attribute name="POPULARITY" value="14" x="-12.7" y="119.38" size="1.778" layer="27" rot="R180" display="off"/>
 <attribute name="VALUE" x="28.575" y="58.42" size="1.27" layer="27" rot="R270"/>
