File: Grupos/2/Review/Motor v2/motor_encoder.sch (EAGLE design)
At the start: 15 parts, among them X1 MKDSN1,5/2-5,08

Commit message: Se finaliza tarjeta grupo 2
Parts:
- added VR1: P160KN, P160KN:P160KN
- C5: device rcl:CPOL-USA -> rcl_v2:CPOL-US
- U1: value (none) -> L9958SB
- X1: value MKDSN1,5/2-5,08 -> 1729128
Connections:
- new net POTE: M1-CN8.PB0, VR1.S
- net GND: now also VR1.CW

Commit message: Se suben archivos posterior a revisión
Parts:
- C1, C2: PARTNO (none) -> GRM2195C1H103JA01D
- C3, C6: PARTNO (none) -> GCM21BR72A104KA37L
- C4: PARTNO (none) -> GCJ219R71C105KA01D
- C5: PARTNO (none) -> EMVE250ADA101MF80G
- R1, R2, R3: PARTNO (none) -> RC0805FR-0710KL
- U1: PARTNO (none) -> L9958SB
- VR1: value P160KN -> P160KN-0QD15B10K; PARTNO (none) -> P160KN-0QD15B10K
- X1: PARTNO (none) -> 1729128
